File: Hardware/BattleBot_Motherboard/BattleBot_Motherboard.kicad_pcb (KiCad board)
At the start: 2 copper layers, 5 parts, among them U1 ESP32-S2-SOLO

Commit message: Getting somewhere?
Parts:
- removed U1: ESP32-S2-SOLO, Espressif:ESP32-S2-SOLO
- added U101: ESP32-S2-SOLO, Espressif:ESP32-S2-SOLO, F.Cu at (141.7, 111.8)
- renumbered H1 to H101, H2 to H102, H3 to H103, H4 to H104
