File: Hardware/BattleBot_Motherboard/BattleBot_Motherboard.kicad_sch (KiCad schematic)
At the start: 6 parts

Commit message: Getting somewhere?
Parts:
- C101: renamed from C?; value (none) -> 0.1uf
- U101: renamed from U1; value (none) -> ESP32-S2-SOLO; footprint (none) -> Espressif:ESP32-S2-SOLO
- renumbered H1 to H101, H2 to H102, H3 to H103, H4 to H104
Changed lines of the file:
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@@
   (symbol (lib_id "power:GND") (at 200.66 114.3 0) (unit 1)
     (in_bom yes) (on_board yes)
-    (property "Reference" "#PWR0101" (id 0) (at 200.66 120.65 0)
-      (effects (font (size 1.27 1.27)) hide)
-    )
-    (property "Value" "" (id 1) (at 200.66 118.11 0))
+    (property "Reference" "#PWR0103" (id 0) (at 200.66 120.65 0)
+      (effects (font (size 1.27 1.27)) hide)
+    )
+    (property "Value" "GND" (id 1) (at 200.66 118.11 0))
     (property "Footprint" "" (id 2) (at 200.66 114.3 0)
       (effects (font (size 1.27 1.27)) hide)
@@
   (symbol (lib_id "Mechanical:MountingHole") (at 19.05 21.59 0) (unit 1)
     (in_bom yes) (on_board yes) (fields_autoplaced)
-    (property "Reference" "H1" (id 0) (at 21.59 20.3199 0)
+    (property "Reference" "H101" (id 0) (at 21.59 20.3199 0)
       (effects (font (size 1.27 1.27)) (justify left))
     )
@@
   (symbol (lib_id "Mechanical:MountingHole") (at 19.05 34.29 0) (unit 1)
     (in_bom yes) (on_board yes) (fields_autoplaced)
-    (property "Reference" "H3" (id 0) (at 21.59 33.0199 0)
+    (property "Reference" "H103" (id 0) (at 21.59 33.0199 0)
       (effects (font (size 1.27 1.27)) (justify left))
     )
@@
   (symbol (lib_id "power:+3.3V") (at 107.95 101.6 0) (unit 1)
     (in_bom yes) (on_board yes)
-    (property "Reference" "#PWR0103" (id 0) (at 107.95 105.41 0)
-      (effects (font (size 1.27 1.27)) hide)
-    )
-    (property "Value" "" (id 1) (at 107.95 97.79 0))
+    (property "Reference" "#PWR0101" (id 0) (at 107.95 105.41 0)
+      (effects (font (size 1.27 1.27)) hide)
+    )
+    (property "Value" "+3.3V" (id 1) (at 107.95 97.79 0))
     (property "Footprint" "" (id 2) (at 107.95 101.6 0)
       (effects (font (size 1.27 1.27)) hide)
@@
   (symbol (lib_id "Device:C_Small") (at 107.95 110.49 0) (unit 1)
     (in_bom yes) (on_board yes)
-    (property "Reference" "C?" (id 0) (at 109.22 109.22 0)
-      (effects (font (size 1.27 1.27)) (justify left))
-    )
-    (property "Value" "" (id 1) (at 109.22 113.03 0)
+    (property "Reference" "C101" (id 0) (at 109.22 109.22 0)
+      (effects (font (size 1.27 1.27)) (justify left))
+    )
+    (property "Value" "0.1uf" (id 1) (at 109.22 113.03 0)
       (effects (font (size 1.27 1.27)) (justify left))
     )
@@
   (symbol (lib_id "Mechanical:MountingHole") (at 19.05 27.94 0) (unit 1)
     (in_bom yes) (on_board yes) (fields_autoplaced)
-    (property "Reference" "H2" (id 0) (at 21.59 26.6699 0)
+    (property "Reference" "H102" (id 0) (at 21.59 26.6699 0)
       (effects (font (size 1.27 1.27)) (justify left))
     )
@@
   (symbol (lib_id "Espressif:ESP32-S2-SOLO") (at 153.67 64.77 0) (unit 1)
     (in_bom yes) (on_board yes) (fields_autoplaced)
-    (property "Reference" "U1" (id 0) (at 153.67 17.78 0))
-    (property "Value" "" (id 1) (at 153.67 20.32 0))
-    (property "Footprint" "" (id 2) (at 153.67 114.3 0)
+    (property "Reference" "U101" (id 0) (at 153.67 17.78 0))
+    (property "Value" "ESP32-S2-SOLO" (id 1) (at 153.67 20.32 0))
+    (property "Footprint" "Espressif:ESP32-S2-SOLO" (id 2) (at 153.67 114.3 0)
       (effects (font (size 1.27 1.27)) hide)
     )
@@
   (symbol (lib_id "Mechanical:MountingHole") (at 19.05 40.64 0) (unit 1)
     (in_bom yes) (on_board yes) (fields_autoplaced)
-    (property "Reference" "H4" (id 0) (at 21.59 39.3699 0)
+    (property "Reference" "H104" (id 0) (at 21.59 39.3699 0)
       (effects (font (size 1.27 1.27)) (justify left))
     )
@@
   )
   (symbol_instances
-    (path "/05219430-e0c9-4db7-944a-06d914af11a5"
-      (reference "#PWR0101") (unit 1) (value "GND") (footprint "")
+    (path "/6f89c48b-e268-40d2-a5d4-4f8eaf2e354e"
+      (reference "#PWR0101") (unit 1) (value "+3.3V") (footprint "")
     )
     (path "/4d93edd4-3fe5-4a85-a849-429789fe23b4"
       (reference "#PWR0102") (unit 1) (value "GND") (footprint "")
     )
-    (path "/6f89c48b-e268-40d2-a5d4-4f8eaf2e354e"
-      (reference "#PWR0103") (unit 1) (value "+3.3V") (footprint "")
+    (path "/05219430-e0c9-4db7-944a-06d914af11a5"
+      (reference "#PWR0103") (unit 1) (value "GND") (footprint "")
     )
     (path "/8b330970-4632-412a-8c11-4d67e7df8c7c"
-      (reference "C?") (unit 1) (value "0.1uf") (footprint "")
+      (reference "C101") (unit 1) (value "0.1uf") (footprint "")
     )
     (path "/1ca854b6-fa72-4706-8d20-31a710f3f33c"
-      (reference "H1") (unit 1) (value "MountingHole") (footprint "MountingHole:MountingHole_2.5mm_Pad")
+      (reference "H101") (unit 1) (value "MountingHole") (footprint "MountingHole:MountingHole_2.5mm_Pad")
     )
     (path "/a397076e-32f4-4b81-aa06-446fc3c851d9"
-      (reference "H2") (unit 1) (value "MountingHole") (footprint "MountingHole:MountingHole_2.5mm_Pad")
+      (reference "H102") (unit 1) (value "MountingHole") (footprint "MountingHole:MountingHole_2.5mm_Pad")
     )
     (path "/51545956-afdd-4ba3-8cf1-1a9677f0be42"
-      (reference "H3") (unit 1) (value "MountingHole") (footprint "MountingHole:MountingHole_2.5mm_Pad")
+      (reference "H103") (unit 1) (value "MountingHole") (footprint "MountingHole:MountingHole_2.5mm_Pad")
     )
     (path "/db284038-3452-455e-8453-88d57db2c118"
-      (reference "H4") (unit 1) (value "MountingHole") (footprint "MountingHole:MountingHole_2.5mm_Pad")
+      (reference "H104") (unit 1) (value "MountingHole") (footprint "MountingHole:MountingHole_2.5mm_Pad")
     )
     (path "/be5f784a-be17-4300-97a7-e317142c7f33"
-      (reference "U1") (unit 1) (value "ESP32-S2-SOLO") (footprint "Espressif:ESP32-S2-SOLO")
-    )
-  )
+      (reference "U101") (unit 1) (value "ESP32-S2-SOLO") (footprint "Espressif:ESP32-S2-SOLO")
+    )
+  )
